Commit message: added suction tool

File: ur_description/urdf/ur5.xacro (robot description, xacro)
@@ -16,3 +16,10 @@
   <xacro:include filename="$(find ur_description)/urdf/inc/ur5_macro.xacro"/>
   <xacro:ur5_robot prefix="" />
+  <xacro:include filename="$(find ur_description)/urdf/inc/suction_tool.xacro"/>
+  <joint name="tool0-suction_tool" type="fixed">
+    <!-- default toolframe: X+ left, Y+ up, Z+ front -->
+    <origin xyz="0 0 0" rpy="0 0 0"/>
+    <parent link="tool0"/>
+    <child link="suction_tool"/>
+  </joint>
 </robot>
