Commit message: change some params for real robot

File: ur_description/urdf/inc/suction_tool.xacro (robot description, xacro)
@@ -20,5 +20,5 @@
     </link>
     <joint name="suction_tool-tool_tip" type="fixed">
-        <origin xyz="0 0 0.16" rpy="0 0 0"/>
+        <origin xyz="0 0 0.178" rpy="0 0 0"/>
         <parent link="suction_tool"/>
         <child link="tool_tip"/>
